File: Schematics/RickNAS_4PortSATA.kicad_pcb (KiCad board)
At the start: 2 copper layers, 122.1 x 69.1 mm, 16 parts, among them U1 SATA_Combined, U10 SATA_Power, U2 SATA_Data, U3 SATA_Power, U4 SATA_Combined, U5 SATA_Data, U6 SATA_Combined, U7 SATA_Data, U8 SATA_Combined, U9 SATA_Data

Commit message: Started CAD
Parts:
- removed kibuzzard-67B4AC38: G***, kibuzzard-67B4AC38
- added D1: LED_Small, LED_SMD:LED_0805_2012Metric, F.Cu at (101.8, 141.2)
- added D2: LED_Small, LED_SMD:LED_0805_2012Metric, F.Cu at (128.8, 141.4)
- added D3: LED_Small, LED_SMD:LED_0805_2012Metric, F.Cu at (155.9, 141.4)
- added D4: LED_Small, LED_SMD:LED_0805_2012Metric, F.Cu at (182.8, 141.4)
- added RN1: R_Pack04, Resistor_SMD:R_Array_Concave_4x0603, F.Cu at (137.8, 134.5)
- added kibuzzard-67B6042A: G***, kibuzzard-67B6042A, F.Cu at (201.8, 108.8)
- added kibuzzard-67B60589: G***, kibuzzard-67B60589, F.Cu at (108.4, 141.2)
- added kibuzzard-67B60597: G***, kibuzzard-67B60597, F.Cu at (135.4, 141.2)
- added kibuzzard-67B605A5: G***, kibuzzard-67B605A5, F.Cu at (162.6, 141.2)
- added kibuzzard-67B605B2: G***, kibuzzard-67B605B2, F.Cu at (189.6, 141.2)
- moved kibuzzard-67B4AC4E 1.51 mm to (205.7, 114.5)
Connections:
- U1 pad 19: VSS -> Drive 1
- U4 pad 19: VSS -> Drive 3
- U6 pad 19: VSS -> Drive 2
- U8 pad 19: VSS -> Drive 4
Routing:
- net Net-(D4-A): track 0.00 -> 48.5 mm
- net Net-(D1-A): track 0.00 -> 37.3 mm
- net +3.3V: track 166.6 -> 198.3 mm
- net Drive 3: track 0.00 -> 29.2 mm, vias 0 -> 2
- net Drive 1: track 0.00 -> 27.0 mm
- net Drive 2: track 0.00 -> 25.7 mm, vias 0 -> 2
- net Drive 4: track 0.00 -> 24.7 mm, vias 0 -> 2
- net Net-(D3-A): track 0.00 -> 22.1 mm
- net Net-(D2-A): track 0.00 -> 11.0 mm
