File: Schematics/V2 - 4 layer PCB/RickNAS_4PortSATA.kicad_pcb (KiCad board)
At the start: 4 copper layers, 32 parts, among them J1 2227595-1, J10 10076579-002C-TRLF, J6 POWER, J7 10076579-002C-TRLF, J8 10076579-002C-TRLF, J9 10076579-002C-TRLF, U1 CH32V003FxPx

Commit message: Progress on V2
Parts:
- moved C9 28.2 mm to (128.4, 82.3)
- moved D2 28.2 mm to (189.0, 78.1)
- moved D4 28.2 mm to (189.0, 84.2)
- moved H1 28.2 mm to (178.9, 62.8)
- moved H3 28.2 mm to (178.9, 77.1)
- moved J1 28.2 mm to (192.8, 102.8)
- moved J10 28.2 mm to (139.3, 75.7)
- moved J6 28.2 mm to (189.9, 63.8)
- moved J8 28.2 mm to (139.3, 55.4)
- moved JP2 28.2 mm to (184.6, 78.9)
- moved JP3 28.2 mm to (184.6, 82.5)
- moved JP3 28.2 mm to (164.7, 45.4)
- moved JP4 28.2 mm to (164.7, 49.0)
- moved RN1 28.2 mm to (193.3, 76.0)
- moved C1 28.2 mm to (133.4, 96.5)
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Changed lines of the file:
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@@
 	(footprint "Jumper:SolderJumper-2_P1.3mm_Open_TrianglePad1.0x1.5mm"
 		(layer "F.Cu")
-		(at 136.5584 51.211599)
+		(at 164.704462 48.971599)
 		(descr "SMD Solder Jumper, 1x1.5mm Triangular Pads, 0.3mm gap, open")
 		(tags "solder jumper open")
@@
 	(footprint "LED_SMD:LED_0805_2012Metric"
 		(layer "F.Cu")
-		(at 160.88 77.345)
+		(at 189.026062 75.105)
 		(descr "LED SMD 0805 (2012 Metric), square (rectangular) end terminal, IPC-7351 nominal, (Body size source: https://docs.google.com/spreadsheets/d/1BsfQQcO9C6DZCsRaXUlFlo91Tg2WpOkGARC1WS5S8t0/edit?usp=sharing), generated with kicad-footprint-generator")
 		(tags "LED")
@@
 	(footprint "Capacitor_THT:CP_Radial_D10.0mm_P5.00mm"
 		(layer "F.Cu")
-		(at 140.668584 110.24)
+		(at 168.814646 108)
 		(descr "CP, Radial series, Radial, pin pitch=5.00mm, diameter=10mm, height=16mm, Electrolytic Capacitor")
 		(tags "CP Radial series Radial pin pitch 5.00mm diameter 10mm height 16mm Electrolytic Capacitor")
@@
 	(footprint "Package_SO:TSSOP-20_4.4x6.5mm_P0.65mm"
 		(layer "F.Cu")
-		(at 93.6834 87.031599)
+		(at 121.829462 84.791599)
 		(descr "TSSOP, 20 Pin (JEDEC MO-153 Var AC https://www.jedec.org/document_search?search_api_views_fulltext=MO-153), generated with kicad-footprint-generator ipc_gullwing_generator.py")
 		(tags "TSSOP SO")
@@
 	(footprint "LED_SMD:LED_0805_2012Metric"
 		(layer "F.Cu")
-		(at 160.88 80.385)
+		(at 189.026062 78.145)
 		(descr "LED SMD 0805 (2012 Metric), square (rectangular) end terminal, IPC-7351 nominal, (Body size source: https://docs.google.com/spreadsheets/d/1BsfQQcO9C6DZCsRaXUlFlo91Tg2WpOkGARC1WS5S8t0/edit?usp=sharing), generated with kicad-footprint-generator")
 		(tags "LED")
@@
 	(footprint "Capacitor_THT:CP_Radial_D10.0mm_P5.00mm"
 		(layer "F.Cu")
-		(at 105.224646 110.24)
+		(at 133.370708 108)
 		(descr "CP, Radial series, Radial, pin pitch=5.00mm, diameter=10mm, height=16mm, Electrolytic Capacitor")
 		(tags "CP Radial series Radial pin pitch 5.00mm diameter 10mm height 16mm Electrolytic Capacitor")
@@
 	(footprint "Capacitor_THT:CP_Radial_D10.0mm_P5.00mm"
 		(layer "F.Cu")
-		(at 140.668584 98.69)
+		(at 168.814646 96.45)
 		(descr "CP, Radial series, Radial, pin pitch=5.00mm, diameter=10mm, height=16mm, Electrolytic Capacitor")
 		(tags "CP Radial series Radial pin pitch 5.00mm diameter 10mm height 16mm Electrolytic Capacitor")
@@
 	(footprint "Jumper:SolderJumper-2_P1.3mm_Open_TrianglePad1.0x1.5mm"
 		(layer "F.Cu")
-		(at 156.46 84.7)
+		(at 184.606062 82.46)
 		(descr "SMD Solder Jumper, 1x1.5mm Triangular Pads, 0.3mm gap, open")
 		(tags "solder jumper open")
@@
 	(footprint "MountingHole:MountingHole_3.2mm_M3_DIN965_Pad"
 		(layer "F.Cu")
-		(at 150.71 79.34)
+		(at 178.856062 77.1)
 		(descr "Mounting Hole 3.2mm, M3, generated by kicad-footprint-generator mountinghole.py")
 		(tags "mountinghole M3 DIN965")
@@
 	(footprint "UE_Connector:CONN_SD-43045-008_04_MOL"
 		(layer "F.Cu")
-		(at 161.7511 66.082599)
+		(at 189.897162 63.842599)
 		(tags "430450423 ")
 		(property "Reference" "J6"
@@
 	(footprint "Jumper:SolderJumper-2_P1.3mm_Open_TrianglePad1.0x1.5mm"
 		(layer "F.Cu")
-		(at 136.5584 44.111599)
+		(at 164.704462 41.871599)
 		(descr "SMD Solder Jumper, 1x1.5mm Triangular Pads, 0.3mm gap, open")
 		(tags "solder jumper open")
@@
 	(footprint "MountingHole:MountingHole_3.2mm_M3_DIN965_Pad"
 		(layer "F.Cu")
-		(at 150.71 65.04)
+		(at 178.856062 62.8)
 		(descr "Mounting Hole 3.2mm, M3, generated by kicad-footprint-generator mountinghole.py")
 		(tags "mountinghole M3 DIN965")
@@
 	(footprint "Jumper:SolderJumper-2_P1.3mm_Open_TrianglePad1.0x1.5mm"
 		(layer "F.Cu")
-		(at 156.46 77.6)
+		(at 184.606062 75.36)
 		(descr "SMD Solder Jumper, 1x1.5mm Triangular Pads, 0.3mm gap, open")
 		(tags "solder jumper open")
@@
 	(footprint "MountingHole:MountingHole_3.2mm_M3_DIN965_Pad"
 		(layer "F.Cu")
-		(at 150.71 86.49)
+		(at 178.856062 84.25)
 		(descr "Mounting Hole 3.2mm, M3, generated by kicad-footprint-generator mountinghole.py")
 		(tags "mountinghole M3 DIN965")
@@
 	(footprint "Capacitor_THT:CP_Radial_D10.0mm_P5.00mm"
 		(layer "F.Cu")
-		(at 117.039292 110.24)
+		(at 145.185354 108)
 		(descr "CP, Radial series, Radial, pin pitch=5.00mm, diameter=10mm, height=16mm, Electrolytic Capacitor")
 		(tags "CP Radial series Radial pin pitch 5.00mm diameter 10mm height 16mm Electrolytic Capacitor")
@@
 	(footprint "Capacitor_THT:CP_Radial_D10.0mm_P5.00mm"
 		(layer "F.Cu")
-		(at 128.853938 98.69)
+		(at 157 96.45)
 		(descr "CP, Radial series, Radial, pin pitch=5.00mm, diameter=10mm, height=16mm, Electrolytic Capacitor")
 		(tags "CP Radial series Radial pin pitch 5.00mm diameter 10mm height 16mm Electrolytic Capacitor")
@@
 	(footprint "Jumper:SolderJumper-2_P1.3mm_Open_TrianglePad1.0x1.5mm"
 		(layer "F.Cu")
-		(at 156.46 81.15)
+		(at 184.606062 78.91)
 		(descr "SMD Solder Jumper, 1x1.5mm Triangular Pads, 0.3mm gap, open")
 		(tags "solder jumper open")
@@
 	(footprint "UE_Connector:22275951"
 		(layer "F.Cu")
-		(at 164.685 105.04)
+		(at 192.831062 102.8)
 		(descr "2227595-1-5")
 		(tags "Connector")
@@
 	(footprint "Capacitor_THT:CP_Radial_D10.0mm_P5.00mm"
 		(layer "F.Cu")
-		(at 128.853938 110.24)
+		(at 157 108)
 		(descr "CP, Radial series, Radial, pin pitch=5.00mm, diameter=10mm, height=16mm, Electrolytic Capacitor")
 		(tags "CP Radial series Radial pin pitch 5.00mm diameter 10mm height 16mm Electrolytic Capacitor")
@@
 	(footprint "Jumper:SolderJumper-2_P1.3mm_Open_TrianglePad1.0x1.5mm"
 		(layer "F.Cu")
-		(at 156.46 88.25)
+		(at 184.606062 86.01)
 		(descr "SMD Solder Jumper, 1x1.5mm Triangular Pads, 0.3mm gap, open")
 		(tags "solder jumper open")
@@
 	(footprint "LED_SMD:LED_0805_2012Metric"
 		(layer "F.Cu")
-		(at 160.88 83.425)
+		(at 189.026062 81.185)
 		(descr "LED SMD 0805 (2012 Metric), square (rectangular) end terminal, IPC-7351 nominal, (Body size source: https://docs.google.com/spreadsheets/d/1BsfQQcO9C6DZCsRaXUlFlo91Tg2WpOkGARC1WS5S8t0/edit?usp=sharing), generated with kicad-footprint-generator")
 		(tags "LED")
@@
 	(footprint "Capacitor_THT:CP_Radial_D10.0mm_P5.00mm"
 		(layer "F.Cu")
-		(at 117.039292 98.69)
+		(at 145.185354 96.45)
 		(descr "CP, Radial series, Radial, pin pitch=5.00mm, diameter=10mm, height=16mm, Electrolytic Capacitor")
 		(tags "CP Radial series Radial pin pitch 5.00mm diameter 10mm height 16mm Electrolytic Capacitor")
@@
 	(footprint "UE_Connector:CONN_10076579-002C-TRLF_AMP"
 		(layer "F.Cu")
-		(at 111.125 47.421299)
+		(at 139.271062 45.181299)
 		(tags "10076579-002C-TRLF ")
 		(property "Reference" "J7"
@@
 	(footprint "UE_Connector:CONN_10076579-002C-TRLF_AMP"
 		(layer "F.Cu")
-		(at 111.125 77.929499)
+		(at 139.271062 75.689499)
 		(tags "10076579-002C-TRLF ")
 		(property "Reference" "J10"
@@
 	(footprint "Resistor_SMD:R_Array_Concave_4x0603"
 		(layer "F.Cu")
-		(at 165.16 78.23)
+		(at 193.306062 75.99)
 		(descr "Thick Film Chip Resistor Array, Wave soldering, Vishay CRA06P (see cra06p.pdf)")
 		(tags "resistor array")
@@
 	(footprint "Capacitor_SMD:C_0805_2012Metric"
 		(layer "F.Cu")
-		(at 100.2784 84.511599)
+		(at 128.424462 82.271599)
 		(descr "Capacitor SMD 0805 (2012 Metric), square (rectangular) end terminal, IPC-7351 nominal, (Body size source: IPC-SM-782 page 76, https://www.pcb-3d.com/wordpress/wp-content/uploads/ipc-sm-782a_amendment_1_and_2.pdf, https://docs.google.com/spreadsheets/d/1BsfQQcO9C6DZCsRaXUlFlo91Tg2WpOkGARC1WS5S8t0/edit?usp=sharing), generated with kicad-footprint-generator")
 		(tags "capacitor")
@@
 	(footprint "LED_SMD:LED_0805_2012Metric"
 		(layer "F.Cu")
-		(at 160.88 86.465)
+		(at 189.026062 84.225)
 		(descr "LED SMD 0805 (2012 Metric), square (rectangular) end terminal, IPC-7351 nominal, (Body size source: https://docs.google.com/spreadsheets/d/1BsfQQcO9C6DZCsRaXUlFlo91Tg2WpOkGARC1WS5S8t0/edit?usp=sharing), generated with kicad-footprint-generator")
 		(tags "LED")
@@
 	(footprint "MountingHole:MountingHole_3.2mm_M3_DIN965_Pad"
 		(layer "F.Cu")
-		(at 150.71 72.19)
+		(at 178.856062 69.95)
 		(descr "Mounting Hole 3.2mm, M3, generated by kicad-footprint-generator mountinghole.py")
 		(tags "mountinghole M3 DIN965")
@@
 	(footprint "Jumper:SolderJumper-2_P1.3mm_Open_TrianglePad1.0x1.5mm"
 		(layer "F.Cu")
-		(at 136.5584 47.661599)
+		(at 164.704462 45.421599)
 		(descr "SMD Solder Jumper, 1x1.5mm Triangular Pads, 0.3mm gap, open")
 		(tags "solder jumper open")
@@
 	(footprint "UE_Connector:CONN_10076579-002C-TRLF_AMP"
 		(layer "F.Cu")
-		(at 111.125 67.760099)
+		(at 139.271062 65.520099)
 		(tags "10076579-002C-TRLF ")
 		(property "Reference" "J9"
@@
 	(footprint "UE_Connector:CONN_10076579-002C-TRLF_AMP"
 		(layer "F.Cu")
-		(at 111.125 57.590699)
+		(at 139.271062 55.350699)
 		(tags "10076579-002C-TRLF ")
 		(property "Reference" "J8"
@@
 	(footprint "Capacitor_THT:CP_Radial_D10.0mm_P5.00mm"
 		(layer "F.Cu")
-		(at 105.224646 98.69)
+		(at 133.370708 96.45)
 		(descr "CP, Radial series, Radial, pin pitch=5.00mm, diameter=10mm, height=16mm, Electrolytic Capacitor")
 		(tags "CP Radial series Radial pin pitch 5.00mm diameter 10mm height 16mm Electrolytic Capacitor")

Commit message: Progress on routing
Parts:
- moved C1 115.7 mm to (20.4, 71.6)
- moved C2 115.7 mm to (20.4, 83.1)
- moved C7 115.7 mm to (55.8, 71.6)
- moved C8 115.7 mm to (55.8, 83.1)
- moved C9 115.7 mm to (15.4, 57.4)
- moved H1 115.7 mm to (65.9, 37.9)
- moved H2 115.7 mm to (65.9, 45.1)
- moved H3 115.7 mm to (65.9, 52.2)
- moved H4 115.7 mm to (65.9, 59.4)
- moved J6 115.7 mm to (76.9, 39.0)
- moved JP1 115.7 mm to (71.6, 50.5)
- moved JP2 115.7 mm to (51.7, 17.0)
- moved JP2 115.7 mm to (71.6, 54.0)
- moved JP3 115.7 mm to (71.6, 57.6)
- moved JP3 115.7 mm to (51.7, 20.6)
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Connections:
- J10 pad P1: Net-(JP4-B) -> Net-(JP1-B)
- J10 pad P2: Net-(JP4-B) -> Net-(JP1-B)
- J10 pad P3: Net-(JP4-B) -> Net-(JP1-B)
- J10 pad S10: unconnected-(J10-PadS10) -> unconnected-(J7-PadS10)
- J10 pad S12: unconnected-(J10-PadS12) -> unconnected-(J7-PadS12)
- J10 pad S13: unconnected-(J10-PadS13) -> unconnected-(J7-PadS13)
- J10 pad S2: /TX3+ -> /TX0+
- J10 pad S3: /TX3- -> /TX0-
- J10 pad S5: /RX3- -> /RX0-
- J10 pad S6: /RX3+ -> /RX0+
- J10 pad S9: unconnected-(J10-PadS9) -> unconnected-(J7-PadS9)
- J8 pad P1: Net-(JP2-B) -> Net-(JP1-B)
- J8 pad P2: Net-(JP2-B) -> Net-(JP1-B)
- J8 pad P3: Net-(JP2-B) -> Net-(JP1-B)
- J8 pad S10: unconnected-(J8-PadS10) -> unconnected-(J7-PadS10)
- J8 pad S12: unconnected-(J8-PadS12) -> unconnected-(J7-PadS12)
- J8 pad S13: unconnected-(J8-PadS13) -> unconnected-(J7-PadS13)
- J8 pad S2: /TX1+ -> /TX0+
- J8 pad S3: /TX1- -> /TX0-
- J8 pad S5: /RX1- -> /RX0-
- J8 pad S6: /RX1+ -> /RX0+
- J8 pad S9: unconnected-(J8-PadS9) -> unconnected-(J7-PadS9)
- J9 pad P1: Net-(JP3-B) -> Net-(JP1-B)
- J9 pad P2: Net-(JP3-B) -> Net-(JP1-B)
- J9 pad P3: Net-(JP3-B) -> Net-(JP1-B)
- J9 pad S10: unconnected-(J9-PadS10) -> unconnected-(J7-PadS10)
- J9 pad S12: unconnected-(J9-PadS12) -> unconnected-(J7-PadS12)
- J9 pad S13: unconnected-(J9-PadS13) -> unconnected-(J7-PadS13)
- J9 pad S2: /TX2+ -> /TX0+
- J9 pad S3: /TX2- -> /TX0-
- J9 pad S5: /RX2- -> /RX0-
- J9 pad S6: /RX2+ -> /RX0+
- J9 pad S9: unconnected-(J9-PadS9) -> unconnected-(J7-PadS9)

Commit message: V2 finished, ordering PCB
Parts:
- removed the JP2 at (71.6, 54.0)
- removed the JP3 at (71.6, 57.6)
- removed the JP4 at (71.6, 61.1)
- added C10: 10uF, Capacitor_SMD:C_0805_2012Metric, F.Cu at (154.4, 36.6)
- added C11: 10uF, Capacitor_SMD:C_0805_2012Metric, F.Cu at (154.4, 39.7)
- added J2: Conn_01x03, Connector_PinHeader_1.00mm:PinHeader_1x03_P1.00mm_Vertical, F.Cu at (166.6, 106.5)
- added J3: Conn_01x03, Connector_PinHeader_2.54mm:PinHeader_1x03_P2.54mm_Vertical, F.Cu at (152.3, 98.6)
- added U2: TLV1117-33, Package_TO_SOT_SMD:SOT-223-3_TabPin2, F.Cu at (148.5, 36.6)
- added kibuzzard-69861090: G***, kibuzzard-69861090, F.Cu at (203.5, 96.2)
- added kibuzzard-6986109D: G***, kibuzzard-6986109D, F.Cu at (186.0, 101.2)
- added kibuzzard-698626E9: G***, kibuzzard-698626E9, F.Cu at (146.9, 101.3)
- C1, C2, C3, C4, C5, C6, C7, C8, J1: moved to B.Cu
- moved H4 181.7 mm to (239.0, 114.5)
- moved JP4 175.1 mm to (221.0, 69.0), turned to 180 degrees
- moved H2 173.5 mm to (239.0, 33.0)
- moved C7 169.1 mm to (223.3, 48.5)
- moved C8 169.1 mm to (223.3, 60.0)
- moved D4 168.8 mm to (237.5, 108.5)
- moved U1 160.2 mm to (161.6, 108.4), turned to 90 degrees
- moved C9 158.2 mm to (163.0, 114.5)
- moved C5 149.6 mm to (191.8, 48.5)
- moved C6 149.6 mm to (191.8, 60.0)
- moved JP3 146.3 mm to (189.8, 69.0), turned to 180 degrees
- moved C1 140.9 mm to (160.8, 60.0)
- moved D3 140.5 mm to (206.5, 108.5)
- moved C3 130.7 mm to (160.8, 48.5)
- moved JP2 119.0 mm to (158.8, 69.0), turned to 180 degrees
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Connections:
- C1 pad 2: GND -> VSS
- C2 pad 2: GND -> VSS
- C3 pad 2: GND -> VSS
- C4 pad 2: GND -> VSS
- C5 pad 2: GND -> VSS
- C6 pad 2: GND -> VSS
- C7 pad 2: GND -> VSS
- C8 pad 2: GND -> VSS
- C9 pad 2: +5V -> +3.3V
- D1 pad 1: Drive 1 -> Net-(D1-K)
- D1 pad 2: Net-(D1-A) -> +3.3V
- D2 pad 1: Drive 2 -> Net-(D2-K)
- D2 pad 2: Net-(D2-A) -> +3.3V
- D3 pad 1: Drive 3 -> Net-(D3-K)
- D3 pad 2: Net-(D3-A) -> +3.3V
- D4 pad 1: Drive 4 -> Net-(D4-K)
- D4 pad 2: Net-(D4-A) -> +3.3V
- J10 pad P1: Net-(JP1-B) -> Net-(JP4-B)
- J10 pad P2: Net-(JP1-B) -> Net-(JP4-B)
- J10 pad P3: Net-(JP1-B) -> Net-(JP4-B)
- J10 pad S10: unconnected-(J7-PadS10) -> unconnected-(J10-PadS10)
- J10 pad S12: unconnected-(J7-PadS12) -> unconnected-(J10-PadS12)
- J10 pad S13: unconnected-(J7-PadS13) -> unconnected-(J10-PadS13)
- J10 pad S2: /TX0+ -> /TX3+
- J10 pad S3: /TX0- -> /TX3-
- J10 pad S5: /RX0- -> /RX3-
- J10 pad S6: /RX0+ -> /RX3+
- J10 pad S9: unconnected-(J7-PadS9) -> unconnected-(J10-PadS9)
- J6 pad 1: GND -> VSS
- J6 pad 2: GND -> VSS
- J8 pad P1: Net-(JP1-B) -> Net-(JP2-B)
- J8 pad P2: Net-(JP1-B) -> Net-(JP2-B)
- J8 pad P3: Net-(JP1-B) -> Net-(JP2-B)
- J8 pad S10: unconnected-(J7-PadS10) -> unconnected-(J8-PadS10)
- J8 pad S12: unconnected-(J7-PadS12) -> unconnected-(J8-PadS12)
- J8 pad S13: unconnected-(J7-PadS13) -> unconnected-(J8-PadS13)
- J8 pad S2: /TX0+ -> /TX1+
- J8 pad S3: /TX0- -> /TX1-
- J8 pad S5: /RX0- -> /RX1-
- J8 pad S6: /RX0+ -> /RX1+
- J8 pad S9: unconnected-(J7-PadS9) -> unconnected-(J8-PadS9)
- J9 pad P1: Net-(JP1-B) -> Net-(JP3-B)
- J9 pad P2: Net-(JP1-B) -> Net-(JP3-B)
- J9 pad P3: Net-(JP1-B) -> Net-(JP3-B)
- J9 pad S10: unconnected-(J7-PadS10) -> unconnected-(J9-PadS10)
- J9 pad S12: unconnected-(J7-PadS12) -> unconnected-(J9-PadS12)
- J9 pad S13: unconnected-(J7-PadS13) -> unconnected-(J9-PadS13)
- J9 pad S2: /TX0+ -> /TX2+
- J9 pad S3: /TX0- -> /TX2-
- J9 pad S5: /RX0- -> /RX2-
- J9 pad S6: /RX0+ -> /RX2+
- J9 pad S9: unconnected-(J7-PadS9) -> unconnected-(J9-PadS9)
- RN1 pad 1: +3.3V -> Net-(D1-K)
- RN1 pad 2: +3.3V -> Net-(D4-K)
- RN1 pad 3: +3.3V -> Net-(D3-K)
- RN1 pad 4: +3.3V -> Net-(D2-K)
- RN1 pad 5: Net-(D1-A) -> Drive 4
- RN1 pad 6: Net-(D2-A) -> Drive 3
- RN1 pad 7: Net-(D3-A) -> Drive 2
- RN1 pad 8: Net-(D4-A) -> Drive 1
- U1 pad 1: unconnected-(U1-PD4-Pad1) -> Drive 1
- U1 pad 10: SClock -> Net-(J2-Pin_1)
- U1 pad 11: SLoad -> Net-(J2-Pin_2)
- U1 pad 12: SDataOut -> Net-(J2-Pin_3)
- U1 pad 13: SDataIn -> SDataOut
- U1 pad 14: unconnected-(U1-PC4-Pad14) -> SDataIn
- U1 pad 15: unconnected-(U1-PC5-Pad15) -> SLoad
- U1 pad 16: unconnected-(U1-PC6-Pad16) -> SClock
- U1 pad 18: unconnected-(U1-PD1-Pad18) -> SWO
- U1 pad 2: unconnected-(U1-PD5-Pad2) -> Drive 2
- U1 pad 3: unconnected-(U1-PD6-Pad3) -> Drive 3
- U1 pad 4: unconnected-(U1-PD7-Pad4) -> Drive 4
- U1 pad 9: +5V -> +3.3V
Routing:
- net +3.3V: track 0.00 -> 307.3 mm, vias 0 -> 4
- net VSS: track 0.00 -> 151.8 mm, vias 0 -> 79
- net Net-(D4-K): track 0.00 -> 84.5 mm
- net /RX0+: track 0.00 -> 57.3 mm, vias 0 -> 1
- net /RX0-: track 0.00 -> 56.2 mm, vias 0 -> 1
- net /TX0+: track 0.00 -> 54.3 mm
- net /TX0-: track 0.00 -> 54.3 mm
- net Net-(D3-K): track 0.00 -> 51.7 mm
- net /TX3+: track 0.00 -> 48.5 mm, vias 0 -> 1
- net /TX3-: track 0.00 -> 48.5 mm, vias 0 -> 1
- net /RX3+: track 0.00 -> 48.3 mm, vias 0 -> 1
- net /RX3-: track 0.00 -> 48.2 mm, vias 0 -> 1
- net SClock: track 0.00 -> 33.3 mm, vias 0 -> 3
- net +12V: track 0.00 -> 28.6 mm, vias 0 -> 12
- net /TX2-: track 0.00 -> 25.8 mm
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- added copper zone on B.Cu, net +12V
- added copper zone on F.Cu, net +5V
- added copper zone on In1.Cu, net VSS
- added copper zone on In2.Cu, net VSS
Other:
- board outline added: 136 x 93 mm
