File: Schematics/V2 - 4 layer PCB/RickNAS_4PortSATA.kicad_pcb (KiCad board)
At the start: 4 copper layers, 136.1 x 56.4 mm, 38 parts, among them J1 2227595-1, J10 10076579-002C-TRLF, J2 Conn_01x03, J3 Conn_01x03, J6 POWER, J7 10076579-002C-TRLF, J8 10076579-002C-TRLF, J9 10076579-002C-TRLF, U1 CH32V003FxPx, U2 TLV1117-33

Commit message: Pemultimate v2 pcb commit
Parts:
- removed J2: Conn_01x03, Connector_PinHeader_1.00mm:PinHeader_1x03_P1.00mm_Vertical
- added D5: LED_Small, LED_SMD:LED_0805_2012Metric, F.Cu at (128.0, 57.8)
- added D6: LED_Small, LED_SMD:LED_0805_2012Metric, F.Cu at (159.3, 57.8)
- added D7: LED_Small, LED_SMD:LED_0805_2012Metric, F.Cu at (190.1, 57.8)
- added D8: LED_Small, LED_SMD:LED_0805_2012Metric, F.Cu at (221.1, 57.8)
- added JP5: P11 GND, Jumper:SolderJumper-2_P1.3mm_Open_TrianglePad1.0x1.5mm, F.Cu at (116.1, 55.8)
- added JP6: P11 GND, Jumper:SolderJumper-2_P1.3mm_Open_TrianglePad1.0x1.5mm, F.Cu at (147.2, 55.8)
- added JP7: P11 GND, Jumper:SolderJumper-2_P1.3mm_Open_TrianglePad1.0x1.5mm, F.Cu at (178.2, 55.8)
- added JP8: P11 GND, Jumper:SolderJumper-2_P1.3mm_Open_TrianglePad1.0x1.5mm, F.Cu at (209.3, 55.8)
- added RN2: 2k, Resistor_SMD:R_Array_Concave_4x0603, F.Cu at (103.8, 88.2)
- added RN3: R_Pack04, Resistor_SMD:R_Array_Concave_4x0603, F.Cu at (95.8, 75.5)
- added kibuzzard-6AAAB169: G***, kibuzzard-6AAAB169, F.Cu at (159.5, 59.8)
- added kibuzzard-6AAAB169: G***, kibuzzard-6AAAB169, F.Cu at (221.5, 59.8)
- added kibuzzard-6AAAB169: G***, kibuzzard-6AAAB169, F.Cu at (128.3, 59.8)
- added kibuzzard-6AAAB169: G***, kibuzzard-6AAAB169, F.Cu at (190.5, 59.8)
- added kibuzzard-6AAAB175: G***, kibuzzard-6AAAB175, F.Cu at (158.9, 64.9)
- added kibuzzard-6AAAB175: G***, kibuzzard-6AAAB175, F.Cu at (220.9, 64.9)
- added kibuzzard-6AAAB175: G***, kibuzzard-6AAAB175, F.Cu at (127.7, 64.9)
- added kibuzzard-6AAAB175: G***, kibuzzard-6AAAB175, F.Cu at (189.9, 64.9)
- J6: value POWER -> Molex 4-pin; footprint UE_Connector:CONN_SD-43045-008_04_MOL -> Connector_TE-Connectivity:TE_MATE-N-LOK_350211-1_1x04_P5.08mm_Vertical; moved to B.Cu
- moved J6 14.6 mm to (163.5, 59.2), turned to 90 degrees
- moved C10 3.83 mm to (131.3, 53.8)
- moved C11 3.83 mm to (133.8, 53.8)
- moved U2 3.83 mm to (131.8, 47.0)
- moved C6 1.71 mm to (178.5, 60.0)
- moved C5 1.71 mm to (178.5, 48.5)
Connections:
- J10 pad P11: VSS -> Net-(JP8-B)
- J10 pad P3: Net-(JP4-B) -> unconnected-(J10-PadP3)
- J6 pad 1: VSS -> +12V
- J6 pad 3: +5V -> VSS
- J6 pad 4: +12V -> +5V
- J7 pad P11: VSS -> Net-(JP5-B)
- J7 pad P3: Net-(JP1-B) -> unconnected-(J7-PadP3)
- J8 pad P11: VSS -> Net-(JP6-B)
- J8 pad P3: Net-(JP2-B) -> unconnected-(J8-PadP3)
- J9 pad P11: VSS -> Net-(JP7-B)
- J9 pad P3: Net-(JP3-B) -> unconnected-(J9-PadP3)
- U1 pad 10: Net-(J2-Pin_1) -> unconnected-(U1-PC0-Pad10)
- U1 pad 11: Net-(J2-Pin_2) -> unconnected-(U1-PC1-Pad11)
- U1 pad 12: Net-(J2-Pin_3) -> unconnected-(U1-PC2-Pad12)
- U1 pad 20: unconnected-(U1-PD3-Pad20) -> /Fault 4
- U1 pad 5: unconnected-(U1-PA1-Pad5) -> /Fault 1
- U1 pad 6: unconnected-(U1-PA2-Pad6) -> /Fault 2
- U1 pad 8: unconnected-(U1-PD0-Pad8) -> /Fault 3
Routing:
- net Net-(D8-K): track 0.00 -> 134.3 mm, vias 0 -> 2
- net Net-(D7-K): track 0.00 -> 104.9 mm, vias 0 -> 2
- net Net-(D6-K): track 0.00 -> 74.2 mm, vias 0 -> 2
- net VSS: track 122.1 -> 179.0 mm
- net Net-(D5-K): track 0.00 -> 42.8 mm, vias 0 -> 2
- net +3.3V: track 247.2 -> 221.5 mm, vias 7 -> 6
- net /Fault 4: track 0.00 -> 14.2 mm, vias 0 -> 2
- net /Fault 3: track 0.00 -> 11.1 mm
- net /Fault 2: track 0.00 -> 8.13 mm
- net Net-(J2-Pin_1): track 7.59 -> 0.00 mm, vias 1 -> 0
- net SLoad: track 72.9 -> 80.4 mm
- net Net-(JP5-B): track 0.00 -> 7.42 mm
- net SClock: track 72.2 -> 79.4 mm
- net /Fault 1: track 0.00 -> 7.15 mm
- net Net-(JP7-B): track 0.00 -> 6.62 mm
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
Commit message: Pemultimate v2 pcb commit
Parts:
- removed kibuzzard-69F8CF71: G***, kibuzzard-69F8CF71
- added kibuzzard-6AAAB40B: G***, kibuzzard-6AAAB40B, B.Cu at (198.1, 79.0)

Commit message: Further cleanup
Parts:
- removed kibuzzard-698626E9: G***, kibuzzard-698626E9
- added kibuzzard-6AAAC547: G***, kibuzzard-6AAAC547, F.Cu at (114.4, 78.0)
Routing:
- net unconnected-(U1-PC0-Pad10): track 1.57 -> 0.00 mm, vias 1 -> 0
- net Net-(JP4-B): track 11.4 -> 10.1 mm
- net Net-(JP3-B): track 7.25 -> 5.98 mm
- net Net-(JP2-B): track 6.42 -> 5.15 mm
- net Net-(JP1-B): track 6.42 -> 5.15 mm
- net Net-(JP5-B): track 7.42 -> 6.58 mm
