File: Schematics/V2 - 4 layer PCB/RickNAS_4PortSATA.kicad_sch (KiCad schematic)
At the start: 34 parts, among them J1 2227595-1, J10 10076579-002C-TRLF, J2 Conn_01x03, J3 Conn_01x03, J6 POWER, J7 10076579-002C-TRLF, J8 10076579-002C-TRLF, J9 10076579-002C-TRLF, U1 CH32V003FxPx, U2 TLV1117-33

Commit message: Rewire J1 to SFF-8643 backplane fixed-end pinout
V1 failed because J1 used the controller pinout on a backplane; SAS
cables are full crossover (SFF-9402 Rev 1.1 Table 8-2).

- J7-J10: drive S2/S3 now on RXn (J1 B/A rows), S6/S5 on TXn (J1 D/C rows)
- J1 sideband: SClock A1, SLoad B1, SDataOut C2, SDataIn D2
- A2 (BP_TYPE) pulled down via R1 4.7k = SGPIO; B2/C1 to VSS; D1 NC
- Note on sheet explaining the pinout

PCB not yet updated from schematic; pairs need rerouting.

Co-Authored-By: Claude Opus 5 <noreply@anthropic.com>
Parts:
- added R1: 4.7k, Resistor_SMD:R_0603_1608Metric, symbol Device:R_Small
Connections:
- net RX0+: now also J7.S2; no longer J7.S6
- net RX0-: now also J7.S3; no longer J7.S5
- net RX1+: now also J8.S2; no longer J8.S6
- net RX1-: now also J8.S3; no longer J8.S5
- net RX2+: now also J9.S2; no longer J9.S6
- net RX2-: now also J9.S3; no longer J9.S5
- net RX3+: now also J10.S2; no longer J10.S6
- net RX3-: now also J10.S3; no longer J10.S5
- net SClock: now also J1.A1 (SB7); no longer J1.A2 (SB0)
- net SDataIn: now also J1.D2 (SB6); no longer J1.D1 (SB5)
- net SDataOut: now also J1.C2 (SB2); no longer J1.C1 (SB4)
- net SLoad: now also J1.B1 (SB3); no longer J1.B2 (SB1)
- net TX0+: now also J7.S6; no longer J7.S2
- net TX0-: now also J7.S5; no longer J7.S3
- net TX1+: now also J8.S6; no longer J8.S2
- net TX1-: now also J8.S5; no longer J8.S3
- net TX2+: now also J9.S6; no longer J9.S2
- net TX2-: now also J9.S5; no longer J9.S3
- net TX3+: now also J10.S6; no longer J10.S2
- net TX3-: now also J10.S5; no longer J10.S3
- net VSS: now also J1.B2 (SB1), J1.C1 (SB4), R1.1
- new net: J1.A2 (SB0), R1.2
- no-connect marks 16 -> 17
Other:
- note added: "J1 = SFF-8643 BACKPLANE fixed-end pinout (SFF-9402 Rev 1.1 Table 8-2). TE symbol pin names are the CONTROLLER names; net names follow SFF-9402 (TX = into cable). Drive S2/S3 (RXn) <- J1 B4/B5,A4/A5,B7/B8,A7/A8; drive S6/S5 (TXn) -> J1 D4/D5,C4/C5,D7/D8,C7/C8. SB0 SClock=A1, SB1 SLoad=B1, SB4 SDataOut=C2, SB5 SDataIn=D2, SB7 BP_TYPE=A2 (R1 pull-down = SGPIO), SB3 GND=B2, SB2 GND=C1, SB6 CNTRLR_TYP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"
