File: Schematics/V2 - 4 layer PCB/RickNAS_4PortSATA.kicad_sch (KiCad schematic)
At the start: 35 parts, among them J1 2227595-1, J10 10076579-002C-TRLF, J2 Conn_01x03, J3 Conn_01x03, J6 POWER, J7 10076579-002C-TRLF, J8 10076579-002C-TRLF, J9 10076579-002C-TRLF, U1 CH32V003FxPx, U2 TLV1117-33

Commit message: Fixed traces
Other:
- note removed: "RXn RXp"
- note removed: "TXp TXn"

Commit message: Re-added traces
Connections:
- net RX2+: now also J10.S2; no longer J9.S2
- net RX2-: now also J10.S3; no longer J9.S3
- net RX3+: now also J9.S2; no longer J10.S2
- net RX3-: now also J9.S3; no longer J10.S3
- net TX2+: now also J10.S6; no longer J9.S6
- net TX2-: now also J10.S5; no longer J9.S5
- net TX3+: now also J9.S6; no longer J10.S6
- net TX3-: now also J9.S5; no longer J10.S5
Other:
- moved on the sheet: J10, J9, JP3, JP4
Changed lines of the file:
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@@
 	(symbol
 		(lib_id "UE-Connector:10076579-002C-TRLF")
-		(at 127 74.93 90)
+		(at 207.01 74.93 90)
 		(unit 1)
 		(body_style 1)
@@
 		(fields_autoplaced yes)
 		(property "Reference" "J9"
-			(at 162.56 57.15 90)
+			(at 242.57 57.15 90)
 			(show_name no)
 			(do_not_autoplace no)
@@
 		)
 		(property "Value" "10076579-002C-TRLF"
-			(at 162.56 59.69 90)
+			(at 242.57 59.69 90)
 			(show_name no)
 			(do_not_autoplace no)
@@
 		)
 		(property "Footprint" "UE_Connector:91908-291512_SAS_Conn"
-			(at 122.936 73.66 0)
+			(at 202.946 73.66 0)
 			(hide yes)
 			(show_name no)
@@
 		)
 		(property "Datasheet" "10076579-002C-TRLF"
-			(at 122.936 74.422 0)
+			(at 202.946 74.422 0)
 			(hide yes)
 			(show_name no)
@@
 		)
 		(property "Description" ""
-			(at 127 74.93 0)
+			(at 207.01 74.93 0)
 			(hide yes)
 			(show_name no)
@@
 	(symbol
 		(lib_id "UE-Connector:10076579-002C-TRLF")
-		(at 207.01 74.93 90)
+		(at 127 74.93 90)
 		(unit 1)
 		(body_style 1)
@@
 		(fields_autoplaced yes)
 		(property "Reference" "J10"
-			(at 242.57 57.15 90)
+			(at 162.56 57.15 90)
 			(show_name no)
 			(do_not_autoplace no)
@@
 		)
 		(property "Value" "10076579-002C-TRLF"
-			(at 242.57 59.69 90)
+			(at 162.56 59.69 90)
 			(show_name no)
 			(do_not_autoplace no)
@@
 		)
 		(property "Footprint" "UE_Connector:91908-291512_SAS_Conn"
-			(at 202.946 73.66 0)
+			(at 122.936 73.66 0)
 			(hide yes)
 			(show_name no)
@@
 		)
 		(property "Datasheet" "10076579-002C-TRLF"
-			(at 202.946 74.422 0)
+			(at 122.936 74.422 0)
 			(hide yes)
 			(show_name no)
@@
 		)
 		(property "Description" ""
-			(at 207.01 74.93 0)
+			(at 127 74.93 0)
 			(hide yes)
 			(show_name no)
@@
 	(symbol
 		(lib_id "Jumper:Jumper_2_Small_Open")
-		(at 165.1 82.55 90)
+		(at 245.11 82.55 90)
 		(unit 1)
 		(body_style 1)
@@
 		(dnp no)
 		(property "Reference" "JP3"
-			(at 162.56 81.28 0)
+			(at 242.57 81.28 0)
 			(show_name no)
 			(do_not_autoplace no)
@@
 		)
 		(property "Value" "open"
-			(at 166.878 80.772 0)
+			(at 246.888 80.772 0)
 			(show_name no)
 			(do_not_autoplace no)
@@
 		)
 		(property "Footprint" "Jumper:SolderJumper-2_P1.3mm_Open_TrianglePad1.0x1.5mm"
-			(at 165.1 82.55 0)
+			(at 245.11 82.55 0)
 			(hide yes)
 			(show_name no)
@@
 		)
 		(property "Datasheet" ""
-			(at 165.1 82.55 0)
+			(at 245.11 82.55 0)
 			(hide yes)
 			(show_name no)
@@
 		)
 		(property "Description" "Jumper, 2-pole, small symbol, open"
-			(at 165.1 82.55 0)
+			(at 245.11 82.55 0)
 			(hide yes)
 			(show_name no)
@@
 	(symbol
 		(lib_id "Jumper:Jumper_2_Small_Open")
-		(at 245.11 82.55 90)
+		(at 165.1 82.55 90)
 		(unit 1)
 		(body_style 1)
@@
 		(dnp no)
 		(property "Reference" "JP4"
-			(at 242.57 81.28 0)
+			(at 162.56 81.28 0)
 			(show_name no)
 			(do_not_autoplace no)
@@
 		)
 		(property "Value" "open"
-			(at 246.888 80.772 0)
+			(at 166.878 80.772 0)
 			(show_name no)
 			(do_not_autoplace no)
@@
 		)
 		(property "Footprint" "Jumper:SolderJumper-2_P1.3mm_Open_TrianglePad1.0x1.5mm"
-			(at 245.11 82.55 0)
+			(at 165.1 82.55 0)
 			(hide yes)
 			(show_name no)
@@
 		)
 		(property "Datasheet" ""
-			(at 245.11 82.55 0)
+			(at 165.1 82.55 0)
 			(hide yes)
 			(show_name no)
@@
 		)
 		(property "Description" "Jumper, 2-pole, small symbol, open"
-			(at 245.11 82.55 0)
+			(at 165.1 82.55 0)
 			(hide yes)
 			(show_name no)

Commit message: Small schematic change
Parts:
- added RN2: R_Pack04, Resistor_THT:R_Array_SIP4, symbol Device:R_Pack04
Connections:
- net +3.3V: now also RN2.5 (R4.2), RN2.6 (R3.2), RN2.7 (R2.2), RN2.8 (R1.2)
- net SClock: now also RN2.1 (R1.1)
- net SDataIn: now also RN2.4 (R4.1)
- net SDataOut: now also RN2.3 (R3.1)
- net SLoad: now also RN2.2 (R2.1)
- net VSS: no longer J10.P11, J7.P11, J8.P11, J9.P11
