File: Schematics/V2 - 4 layer PCB/RickNAS_4PortSATA.kicad_sch (KiCad schematic)
At the start: 36 parts, among them J1 2227595-1, J10 10076579-002C-TRLF, J2 Conn_01x03, J3 Conn_01x03, J6 POWER, J7 10076579-002C-TRLF, J8 10076579-002C-TRLF, J9 10076579-002C-TRLF, U1 CH32V003FxPx, U2 TLV1117-33

Commit message: Molex power input, P11 GND jumpers, split P3, drop J2
- J6: 2x2 Micro-Fit -> 4-pin PC peripheral power header (TE MATE-N-LOK
  350211-1 footprint; MPN HC-C5080-4AS / LCSC C5221226). Pins 1=+12V,
  2=GND, 3=GND, 4=+5V. Micro-Fit's 5 A contact was below 4-drive spin-up.
- P11 on J7-J10 through open solder jumpers JP5-JP8 to VSS (default
  floating = staggered spin-up; bridge for immediate spin-up).
- P3 (PWDIS) split off the P1/P2 3.3V bracket on all drives, now NC, so
  closing JP1-JP4 no longer holds drives in power-disable.
- J2 removed; U1 PC0-PC2 marked no-connect.
- RN2 (SGPIO 2k pull-ups, SFF-8485 6.2): value 2k, footprint
  R_Array_Concave_4x0603 (was 4-pad SIP4 on an 8-pin symbol).

PCB not updated; verify J6 pin 1 vs the physical plug before ordering.

Co-Authored-By: Claude Opus 5 <noreply@anthropic.com>
Parts:
- removed J2: Conn_01x03, Connector_PinHeader_1.00mm:PinHeader_1x03_P1.00mm_Vertical, symbol Connector_Generic:Conn_01x03
- added JP5, JP6, JP7, JP8: P11 GND, Jumper:SolderJumper-2_P1.3mm_Open_TrianglePad1.0x1.5mm, symbol Jumper:Jumper_2_Small_Open
- J6: value POWER -> Molex 4-pin; footprint UE_Connector:CONN_SD-43045-008_04_MOL -> Connector_TE-Connectivity:TE_MATE-N-LOK_350211-1_1x04_P5.08mm_Vertical; symbol molex_microfit_2x2:430450423 -> Connector_Generic:Conn_01x04; LCSC (none) -> C5221226; MPN (none) -> HC-C5080-4AS
- RN2: value R_Pack04 -> 2k; footprint Resistor_THT:R_Array_SIP4 -> Resistor_SMD:R_Array_Concave_4x0603
Connections:
- net +12V: now also J6.1 (Pin_1); no longer J6.4
- net +5V: now also J6.4 (Pin_4); no longer J6.3
- net VSS: now also J6.3 (Pin_3), JP5.1 (A), JP6.1 (A), JP7.1 (A), JP8.1 (A); no longer J6.1
- net at J9.P1, J9.P2, JP3.2 (B): no longer J9.P3
- net at J9.P11: now also JP7.2 (B)
- net at J8.P1, J8.P2, JP2.2 (B): no longer J8.P3
- net at J8.P11: now also JP6.2 (B)
- net at J10.P1, J10.P2, JP4.2 (B): no longer J10.P3
- net at J10.P11: now also JP8.2 (B)
- net at J7.P1, J7.P2, JP1.2 (B): no longer J7.P3
- net at J7.P11: now also JP5.2 (B)
- no-connect marks 17 -> 24
