File: Schematics/V2 - 4 layer PCB/RickNAS_4PortSATA.kicad_sch (KiCad schematic)
At the start: 39 parts, among them J1 2227595-1, J10 10076579-002C-TRLF, J3 Conn_01x03, J6 Molex 4-pin, J7 10076579-002C-TRLF, J8 10076579-002C-TRLF, J9 10076579-002C-TRLF, U1 CH32V003FxPx, U2 TLV1117-33

Commit message: Pemultimate v2 pcb commit
Parts:
- added D5, D6, D7, D8: LED_Small, LED_SMD:LED_0805_2012Metric, symbol Device:LED_Small
- added RN3: R_Pack04, Resistor_SMD:R_Array_Concave_4x0603, symbol Device:R_Pack04
Connections:
- net +3.3V: now also D5.2 (A), D6.2 (A), D7.2 (A), D8.2 (A)
- net SClock: now also RN2.4 (R4.1); no longer RN2.1 (R1.1)
- net SDataIn: now also RN2.1 (R1.1); no longer RN2.4 (R4.1)
- net SDataOut: now also RN2.2 (R2.1); no longer RN2.3 (R3.1)
- net SLoad: now also RN2.3 (R3.1); no longer RN2.2 (R2.1)
- net Fault 4: now reaches U1.20 (PD3)
- net Fault 4: now also RN3.5 (R4.2)
- net Fault 1: now reaches U1.5 (PA1)
- net Fault 1: now also RN3.8 (R1.2)
- net Fault 2: now reaches U1.6 (PA2)
- net Fault 2: now also RN3.7 (R2.2)
- net Fault 3: now reaches U1.8 (PD0)
- net Fault 3: now also RN3.6 (R3.2)
- new net: D7.1 (K), RN3.2 (R2.1)
- new net: D5.1 (K), RN3.4 (R4.1)
- new net: D6.1 (K), RN3.3 (R3.1)
- new net: D8.1 (K), RN3.1 (R1.1)
Other:
- moved on the sheet: J6, RN2
